File: BioHackBoardPolulu.brd (EAGLE design)
At the start: 69.5 x 53.5 mm, 42 parts, among them J10 CON_HEADER_1X02-PTH, J11 CON_HEADER_1X02-PTH, J12 CON_HEADER_1X02-PTH, J13 JUMPER_SOLDER_1X2, J2 8x1F-H8.5, J3 8x1F-H8.5, J4 6x1F-H8.5, J7 CON_HEADER_1X02-PTH, J8 CON_HEADER_1X02-PTH, J9 CON_HEADER_1X02-PTH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

Commit message: * Biohackboard version that's shipped.
Parts:
- JP3: value (none) -> 8x1F-H8.5
- Q1, Q2: value IRF512 -> IRF520
Other:
- board text added: "+"
- board text added: "-"
- board text added: "D5"
- board text added: "D6"
Changed lines of the file:
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@@
 <wire x1="35.9" y1="17.9" x2="35.9" y2="16" width="0.4064" layer="21"/>
 <wire x1="35.9" y1="16" x2="36" y2="16" width="0.4064" layer="21"/>
-<text x="55.6" y="15.9" size="1.27" layer="21" rot="R90">GND</text>
-<text x="56.1" y="41.7" size="1.27" layer="21" rot="R90">GND</text>
-<text x="61.4" y="36.8" size="1.27" layer="21" rot="R90">GND</text>
-<text x="61.5" y="26" size="1.27" layer="21" rot="R90">GND</text>
-<text x="61.2" y="21.4" size="1.27" layer="21" rot="R90">V+</text>
-<text x="61.4" y="32.6" size="1.27" layer="21" rot="R90">V+</text>
+<text x="62.9025" y="23.8375" size="1.27" layer="21" rot="R90">D6</text>
+<text x="62.45" y="35.0325" size="1.27" layer="21" rot="R90">D5</text>
+<text x="61.0825" y="39.0225" size="1.27" layer="21" rot="R90">-</text>
+<text x="61.1825" y="28.2225" size="1.27" layer="21" rot="R90">-</text>
+<text x="61.5175" y="20.765" size="1.27" layer="21" rot="R90">+</text>
+<text x="61.0825" y="32.6" size="1.27" layer="21" rot="R90">+</text>
 <text x="63" y="16.2" size="1.27" layer="21" rot="R90">V+</text>
 <text x="63" y="43" size="1.27" layer="21" rot="R90">V+</text>
@@
 <text x="-1.27" y="38.735" size="1.016" layer="21" rot="R180">DIR</text>
 <text x="-0.9525" y="20.955" size="1.016" layer="21" rot="R180">GND</text>
+<text x="56.0025" y="43.4675" size="1.27" layer="21" rot="R90">-</text>
+<text x="56.0025" y="16.7975" size="1.27" layer="21" rot="R90">-</text>
 </plain>
 <attributes>
@@
 <attribute name="VALUE" x="53.442" y="13.6494" size="1.27" layer="27" rot="R270"/>
 </element>
-<element name="JP3" library="pinhead-2" package="1X08-S" value="" x="10.766" y="50.8" smashed="yes">
+<element name="JP3" library="pinhead-2" package="1X08-S" value="8x1F-H8.5" x="10.766" y="50.8" smashed="yes">
 <attribute name="VALUE" x="0.606" y="47.625" size="1.27" layer="27"/>
 </element>
@@
 <attribute name="VALUE" x="11.43" y="19.431" size="1.27" layer="27" rot="R180"/>
 </element>
-<element name="Q1" library="transistor-power" package="TO220BV" value="IRF512" x="46.7388" y="36.6616" smashed="yes" rot="R270"/>
-<element name="Q2" library="transistor-power" package="TO220BV" value="IRF512" x="46.688" y="24.9776" smashed="yes" rot="R270"/>
+<element name="Q1" library="transistor-power" package="TO220BV" value="IRF520" x="46.7388" y="36.6616" smashed="yes" rot="R270"/>
+<element name="Q2" library="transistor-power" package="TO220BV" value="IRF520" x="46.688" y="24.9776" smashed="yes" rot="R270"/>
 <element name="R1" library="SmartPrj" package="R0603-ROUND" value="220" x="37.7952" y="44.564" smashed="yes" rot="R180">
 <attribute name="VALUE" x="37.4158" y="45.604" size="0.8128" layer="27" font="vector"/>
@@
 </element>
 <element name="RENC2" library="pinhead-2" package="1X03-S" value="" x="47.799" y="12.311" smashed="yes" rot="R90">
-<attribute name="NAME" x="45.9702" y="9.6948" size="1.27" layer="25" ratio="10" rot="R90"/>
 <attribute name="VALUE" x="50.974" y="9.771" size="1.27" layer="27" rot="R90"/>
 </element>
